File: PCB/Temp/PCB_1.2/PCB_Gabri1.1.1.brd (EAGLE design)
At the start: 40 x 22 mm, 10 parts, among them U1 VEML6030, U2 TXS0104ED, X1 0446200002

Commit message: PCB drawings
Parts:
- removed C3, C4: (no value), resistor:C025-024X044
- moved R3 4.51 mm to (90.5, 63.0)
- moved R1 1.50 mm to (86.7, 67.9)
- moved D1 0.85 mm to (80.4, 61.4)
- moved U1 0.74 mm to (80.3, 65.2)
- moved C2 0.60 mm to (84.9, 63.1)
- moved C1 0.41 mm to (88.0, 63.1)
Connections:
- net GND: no longer C3.2, C4.2
- net VCCA: no longer C3.1
- net VCCB: no longer C4.1
Routing:
- net SCL: track 0.00 -> 22.0 mm, vias 0 -> 2
- net VCCB: track 33.9 -> 15.7 mm
- net LS_VDD: track 27.2 -> 11.8 mm
- net SDA: track 0.00 -> 10.1 mm
- net INT: track 0.00 -> 9.61 mm
- net LED_1: track 17.0 -> 13.3 mm
- net VCCA: track 41.5 -> 39.3 mm, vias 1 -> 3
- net A3: track 39.5 -> 37.8 mm
- net A1: track 36.2 -> 34.9 mm
- net LED_2: track 11.6 -> 10.7 mm
- net A2: track 45.2 -> 44.3 mm
- removed copper zone on layer 1, net GND
- removed copper zone on layer 16, net GND
