File: PCB/Temp/PCB_1.2/PCB_Gabri1.1.brd (EAGLE design)
At the start: 40 x 22 mm, 10 parts, among them U1 VEML6030, U2 TXS0104ED, X1 0446200002

Commit message: PCB drawings
Parts:
- removed C3, C4: (no value), resistor:C025-024X044
- moved C2 11.0 mm to (94.3, 69.9), turned to 0 degrees
- moved R1 10.8 mm to (95.1, 63.8)
- moved C1 7.15 mm to (94.3, 67.0), turned to 0 degrees
- moved D1 4.97 mm to (85.5, 64.1), turned to 90 degrees
- moved R3 3.61 mm to (89.3, 64.0), turned to 270 degrees
- moved U1 1.10 mm to (81.8, 64.2), turned to 90 degrees
Connections:
- net GND: no longer C3.2, C4.2
- net VCCA: no longer C3.1
- net VCCB: no longer C4.1
Routing:
- net INT: track 0.00 -> 15.7 mm
- net SDA: track 0.00 -> 14.9 mm
- net SCL: track 0.00 -> 13.6 mm
- net VCCB: track 33.9 -> 26.1 mm, vias 0 -> 1
- net LED_2: track 11.6 -> 3.90 mm
- net LS_VDD: track 27.2 -> 30.0 mm, vias 0 -> 2
- net LED_1: track 17.0 -> 15.0 mm, vias 0 -> 1
- net VCCA: track 41.5 -> 39.8 mm, vias 1 -> 3
- net A3: track 39.5 -> 37.8 mm
- net A1: track 36.2 -> 34.9 mm
- net A2: track 45.2 -> 44.3 mm
- removed copper zone on layer 1, net GND
- removed copper zone on layer 16, net GND
Other:
- board size 40 x 22 mm -> 39.4 x 22 mm
