File: PCB/Models/PCB_1/PCB_Gabri1.1.1.brd (EAGLE design)
At the start: 40 x 22 mm, 10 parts, among them U1 VEML6030, U2 TXS0104ED, X1 0446200002

Commit message: PCB drawings
Parts:
- moved C2 11.0 mm to (85.3, 63.5), turned to 270 degrees
- moved R1 10.8 mm to (85.3, 68.5)
- moved C1 7.15 mm to (88.1, 63.5), turned to 270 degrees
- moved D1 4.97 mm to (81.2, 61.7), turned to 0 degrees
- moved R3 3.61 mm to (90.2, 67.5), turned to 90 degrees
- moved U1 1.36 mm to (80.7, 65.0), turned to 0 degrees
Routing:
- net LS_VDD: track 32.0 -> 11.8 mm, vias 2 -> 0
- net VCCB: track 32.9 -> 19.8 mm, vias 1 -> 0
- net LED_1: track 16.5 -> 7.57 mm, vias 1 -> 0
- net SCL: track 15.0 -> 23.3 mm, vias 0 -> 2
- net INT: track 16.6 -> 10.1 mm
- net LED_2: track 5.80 -> 11.6 mm
- net SDA: track 15.8 -> 10.8 mm
Other:
- board size 40 x 22 mm -> 35 x 22.4 mm

Commit message: just a few changes
Routing:
- net A1: track 36.2 -> 32.7 mm
- net GND: track 0.83 -> 2.99 mm
- net A3: track 39.5 -> 40.5 mm
Other:
- board size 35 x 22.4 mm -> 35 x 22 mm
Changed lines of the file:
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@@
 <board>
 <plain>
-<wire x1="59.95" y1="59.65" x2="94.9" y2="59.7" width="0" layer="20"/>
-<wire x1="94.9" y1="59.7" x2="94.85" y2="82" width="0" layer="20"/>
-<wire x1="94.85" y1="82" x2="60" y2="82" width="0" layer="20"/>
-<wire x1="60" y1="82" x2="59.95" y2="59.65" width="0" layer="20"/>
-<dimension x1="100" y1="82" x2="60" y2="82" x3="80" y3="84.6" textsize="1.778" layer="16" dtype="horizontal"/>
-<dimension x1="60" y1="82" x2="60" y2="60" x3="57.2" y3="71" textsize="1.778" layer="16" dtype="horizontal"/>
-<dimension x1="60" y1="82" x2="100" y2="82" x3="80" y3="84.1" textsize="1.778" layer="1"/>
-<dimension x1="100" y1="82" x2="100" y2="60" x3="104.1" y3="71" textsize="1.778" layer="1"/>
-<dimension x1="59.95" y1="59.65" x2="94.9" y2="59.7" x3="77.431678125" y3="55.005409375" textsize="1.778" layer="1"/>
-<dimension x1="60" y1="82" x2="59.95" y2="59.65" x3="54.90421875" y3="70.83634375" textsize="1.778" layer="1"/>
+<wire x1="60" y1="60" x2="95" y2="60" width="0" layer="20"/>
+<wire x1="95" y1="60" x2="95" y2="82" width="0" layer="20"/>
+<wire x1="95" y1="82" x2="60" y2="82" width="0" layer="20"/>
+<wire x1="60" y1="82" x2="60" y2="60" width="0" layer="20"/>
 </plain>
 <attributes>
@@
 <contactref element="U2" pad="2"/>
 <contactref element="X1" pad="1"/>
-<wire x1="66.9" y1="70.8" x2="66.3" y2="70.8" width="0.3048" layer="1"/>
-<wire x1="66.3" y1="70.8" x2="64.2" y2="70.8" width="0.3048" layer="1"/>
-<wire x1="64.2" y1="70.8" x2="63.3" y2="71.7" width="0.3048" layer="1"/>
-<wire x1="63.3" y1="71.7" x2="63.3" y2="73.5" width="0.3048" layer="1"/>
-<wire x1="75.9" y1="79.2" x2="76" y2="79.2" width="0.3048" layer="1"/>
-<wire x1="76" y1="79.2" x2="82.8" y2="79.2" width="0.3048" layer="1"/>
-<wire x1="87.6" y1="73.8" x2="82.8" y2="79.2" width="0.3048" layer="1"/>
-<wire x1="66.3" y1="70.8" x2="67.3494" y2="70.8" width="0.3048" layer="1"/>
-<wire x1="67.3494" y1="70.8" x2="67.3894" y2="70.76" width="0.3048" layer="1"/>
-<wire x1="87.376" y1="73.66" x2="87.516" y2="73.8" width="0.3048" layer="1"/>
-<wire x1="87.516" y1="73.8" x2="87.6" y2="73.8" width="0.3048" layer="1"/>
-<wire x1="63.3" y1="73.5" x2="69" y2="79.2" width="0.3048" layer="1"/>
-<wire x1="69" y1="79.2" x2="75.9" y2="79.2" width="0.3048" layer="1"/>
+<wire x1="67.3894" y1="70.76" x2="65.29" y2="70.76" width="0.3048" layer="1"/>
+<wire x1="65.29" y1="70.76" x2="64.4" y2="71.65" width="0.3048" layer="1"/>
+<wire x1="64.4" y1="71.65" x2="64.4" y2="73.65" width="0.3048" layer="1"/>
+<wire x1="64.4" y1="73.65" x2="69.65" y2="78.9" width="0.3048" layer="1"/>
+<wire x1="69.65" y1="78.9" x2="82.136" y2="78.9" width="0.3048" layer="1"/>
+<wire x1="82.136" y1="78.9" x2="87.376" y2="73.66" width="0.3048" layer="1"/>
 </signal>
 <signal name="A2">
 <contactref element="X1" pad="2"/>
 <contactref element="U2" pad="3"/>
-<wire x1="64.5" y1="69.3" x2="65.8" y2="69.3" width="0.3048" layer="1"/>
-<wire x1="64.5" y1="69.3" x2="62.4" y2="71.4" width="0.3048" layer="1"/>
-<wire x1="62.4" y1="71.4" x2="62.4" y2="73.8" width="0.3048" layer="1"/>
-<wire x1="75.6" y1="80.1" x2="75.7" y2="80.1" width="0.3048" layer="1"/>
-<wire x1="75.7" y1="80.1" x2="83.4" y2="80.1" width="0.3048" layer="1"/>
+<wire x1="68.7" y1="80.1" x2="83.4" y2="80.1" width="0.3048" layer="1"/>
 <wire x1="83.4" y1="80.1" x2="89.1" y2="73.8" width="0.254" layer="1"/>
 <wire x1="89.1" y1="73.8" x2="89.1" y2="72.3" width="0.3048" layer="1"/>
 <wire x1="89.1" y1="72.3" x2="88.5" y2="71.7" width="0.3048" layer="1"/>
 <wire x1="86.4" y1="71.7" x2="88.5" y2="71.7" width="0.3048" layer="1"/>
-<wire x1="65.8" y1="69.3" x2="67.3894" y2="69.3" width="0.3048" layer="1"/>
+<wire x1="67.3894" y1="69.3" x2="64.5" y2="69.3" width="0.3048" layer="1"/>
 <wire x1="67.3894" y1="69.3" x2="67.3894" y2="69.49" width="0.3048" layer="1"/>
 <wire x1="86.36" y1="71.882" x2="86.4" y2="71.842" width="0.3048" layer="1"/>
 <wire x1="86.4" y1="71.842" x2="86.4" y2="71.7" width="0.3048" layer="1"/>
-<wire x1="62.4" y1="73.8" x2="68.7" y2="80.1" width="0.3048" layer="1"/>
-<wire x1="68.7" y1="80.1" x2="75.6" y2="80.1" width="0.3048" layer="1"/>
+<wire x1="64.5" y1="69.3" x2="63" y2="70.8" width="0.3048" layer="1"/>
+<wire x1="63" y1="70.8" x2="63" y2="74.4" width="0.3048" layer="1"/>
+<wire x1="63" y1="74.4" x2="68.7" y2="80.1" width="0.3048" layer="1"/>
 </signal>
 <signal name="A3">
 <contactref element="U2" pad="4"/>
 <contactref element="X1" pad="3"/>
-<wire x1="66.6" y1="68.1" x2="66" y2="68.1" width="0.3048" layer="1"/>
-<wire x1="66" y1="68.1" x2="64.5" y2="68.1" width="0.3048" layer="1"/>
-<wire x1="64.5" y1="68.1" x2="61.5" y2="71.1" width="0.3048" layer="1"/>
-<wire x1="61.5" y1="71.1" x2="61.5" y2="74.1" width="0.3048" layer="1"/>
-<wire x1="61.5" y1="74.1" x2="66.5" y2="79.2" width="0.3048" layer="1"/>
-<via x="66.5" y="79.2" extent="1-16" drill="0.6"/>
-<wire x1="80.4" y1="79.2" x2="85.5" y2="73.8" width="0.4064" layer="16"/>
-<wire x1="66" y1="68.1" x2="66.12" y2="68.22" width="0.3048" layer="1"/>
-<wire x1="66.12" y1="68.22" x2="67.3894" y2="68.22" width="0.3048" layer="1"/>
+<via x="64.9" y="79.2" extent="1-16" drill="0.6"/>
+<wire x1="85.5" y1="73.8" x2="80.4" y2="79.2" width="0.4064" layer="16"/>
 <wire x1="85.344" y1="73.66" x2="85.484" y2="73.8" width="0.3048" layer="16"/>
 <wire x1="85.484" y1="73.8" x2="85.5" y2="73.8" width="0.3048" layer="16"/>
-<wire x1="66.5" y1="79.2" x2="80.4" y2="79.2" width="0.3048" layer="16"/>
+<wire x1="61.5" y1="75.8" x2="64.9" y2="79.2" width="0.3048" layer="1"/>
+<wire x1="80.4" y1="79.2" x2="64.9" y2="79.2" width="0.3048" layer="16"/>
+<wire x1="67.3894" y1="68.22" x2="63.08" y2="68.22" width="0.3048" layer="1"/>
+<wire x1="63.08" y1="68.22" x2="61.5" y2="69.8" width="0.3048" layer="1"/>
+<wire x1="61.5" y1="69.8" x2="61.5" y2="75.8" width="0.3048" layer="1"/>
 </signal>
 <signal name="VCCA">
@@
 <contactref element="U1" pad="3"/>
 <contactref element="U2" pad="11"/>
-<wire x1="79.825" y1="64.3" x2="78.95" y2="64.3" width="0.3048" layer="1"/>
-<wire x1="77.35" y1="65.9" x2="77.35" y2="67.25" width="0.3048" layer="1"/>
-<wire x1="77.35" y1="67.25" x2="76.63" y2="68.22" width="0.3048" layer="1"/>
-<wire x1="76.63" y1="68.22" x2="72.19" y2="68.22" width="0.3048" layer="1"/>
-<wire x1="78.95" y1="64.3" x2="77.35" y2="65.9" width="0.3048" layer="1"/>
+<wire x1="72.19" y1="68.22" x2="76.93" y2="68.22" width="0.3048" layer="1"/>
+<wire x1="77.892" y1="67.258" x2="77.892" y2="65.639575" width="0.3048" layer="1"/>
+<wire x1="77.892" y1="65.639575" x2="79.089575" y2="64.442" width="0.3048" layer="1"/>
+<wire x1="79.089575" y1="64.442" x2="79.108" y2="64.442" width="0.3048" layer="1"/>
+<wire x1="79.108" y1="64.442" x2="79.25" y2="64.3" width="0.3048" layer="1"/>
+<wire x1="76.93" y1="68.22" x2="77.892" y2="67.258" width="0.3048" layer="1"/>
+<wire x1="79.25" y1="64.3" x2="79.825" y2="64.3" width="0.3048" layer="1"/>
 </signal>
 <signal name="SDA">
@@
 <wire x1="72.19" y1="69.49" x2="73.51" y2="69.49" width="0.3048" layer="1"/>
 <wire x1="73.51" y1="69.49" x2="74.1" y2="68.9" width="0.3048" layer="1"/>
-<wire x1="74.1" y1="68.9" x2="77.6" y2="68.9" width="0.3048" layer="1"/>
-<wire x1="77.6" y1="68.9" x2="78.4" y2="67.85" width="0.3048" layer="1"/>
-<wire x1="78.4" y1="67.85" x2="78.4" y2="65.85" width="0.3048" layer="1"/>
 <wire x1="78.4" y1="65.85" x2="79.3" y2="64.95" width="0.3048" layer="1"/>
 <wire x1="79.3" y1="64.95" x2="79.825" y2="64.95" width="0.3048" layer="1"/>
+<wire x1="74.1" y1="68.9" x2="77.35" y2="68.9" width="0.3048" layer="1"/>
+<wire x1="77.35" y1="68.9" x2="78.4" y2="67.85" width="0.3048" layer="1"/>
+<wire x1="78.4" y1="67.85" x2="78.4" y2="65.85" width="0.3048" layer="1"/>
 </signal>
 <signal name="GND">
@@
 <contactref element="U2" pad="5"/>
 <contactref element="X1" pad="8"/>
-<polygon width="0.3048" layer="1">
-<vertex x="60.1" y="81.7"/>
-<vertex x="99.6" y="81.7"/>
-<vertex x="99.6" y="60.4"/>
-<vertex x="60.5" y="60.4"/>
-<vertex x="60.5" y="60.9"/>
-</polygon>
-<polygon width="0.3048" layer="16">
-<vertex x="60.5" y="81.6"/>
-<vertex x="99.6" y="81.6"/>
-<vertex x="99.6" y="60.2"/>
-<vertex x="60.2" y="60.2"/>
-<vertex x="60.2" y="62.2"/>
-<vertex x="60.2" y="81.7"/>
-<vertex x="60.3" y="81.7"/>
-</polygon>
 <via x="65.5" y="66.9" extent="1-16" drill="0.35"/>
 <via x="65.5" y="64.4" extent="1-16" drill="0.35"/>
@@
 <wire x1="82.95" y1="64.1" x2="82.4056" y2="64.1" width="0.3048" layer="1"/>
 <wire x1="82.4056" y1="64.1" x2="82.2056" y2="64.3" width="0.3048" layer="1"/>
+<wire x1="72.19" y1="66.95" x2="74.25" y2="66.95" width="0.1524" layer="1"/>
+<wire x1="74.25" y1="66.95" x2="74.25" y2="67.05" width="0.1524" layer="1"/>
+<polygon width="0.1524" layer="16">
+<vertex x="60.25" y="81.75"/>
+<vertex x="60.25" y="60.35"/>
+<vertex x="94.7" y="60.35"/>
+<vertex x="94.7" y="81.75"/>
+</polygon>
+<polygon width="0.1524" layer="1">
+<vertex x="60.25" y="81.75"/>
+<vertex x="94.7" y="81.75"/>
+<vertex x="94.7" y="60.35"/>
+<vertex x="60.25" y="60.35"/>
+<vertex x="60.25" y="81.7"/>
+</polygon>
 </signal>
 <signal name="LED_1">

Commit message: Update
Parts:
- moved R3 1.92 mm to (92.0, 68.0)
- moved C1 1.47 mm to (89.5, 63.7)
- moved C2 1.27 mm to (86.5, 63.7)
- moved C3 0.50 mm to (62.8, 65.2)
Routing:
- net LED_2: track 11.6 -> 15.5 mm
- net VCCA: track 41.5 -> 38.0 mm
- net GND: track 2.99 -> 6.03 mm, vias 3 -> 4
- net SCL: track 23.3 -> 26.1 mm
- net LED_1: track 7.57 -> 9.21 mm
- net VCCB: track 19.8 -> 18.4 mm
- net SDA: track 10.7 -> 9.52 mm
