File: PCB/Models/PCB_2/PCB_2.1.brd (EAGLE design)
At the start: 35 x 22 mm, 10 parts, among them U1 VEML6030, U2 TXS0104ED, X1 0446200002

Commit message: just a few changes
Parts:
- removed C1, C2, C3, C4: (no value), resistor:C025-024X044
- removed D1: 5988170107F, 5988170107F:LEDC2012X70N
- removed U1: VEML6030, VEML6030:VISHAY_VEML6030_2X2X0.87
- removed U2: TXS0104ED, TXS0104ED:SOIC127P600X175-14N
- added R2: (no value), resistor:R0805
- added SV1: (no value), con-lsta:FE20-2
- added U3: TXS0104ED, TXS0104ED:SOIC127P600X175-14N
- moved X1 103.7 mm to (3.81, 10.2), flipped to the top, turned to 270 degrees
- moved R3 82.0 mm to (34.3, 7.62), turned to 0 degrees
- moved R1 72.0 mm to (34.3, 17.8), turned to 180 degrees
Connections:
- removed net LED_1: R3.2, X1.4
- removed net LED_2: D1.A, R3.1
- removed net LS_VDD: C1.1, C2.1, R1.2, U1.6
- new net LED: R3.1, X1.4
- new net N$1: R3.2, SV1.37
- new net OE: U3.8
- net A1: now also U3.2; no longer U2.2
- net A2: now also U3.3; no longer U2.3
- net A3: now also U3.4; no longer U2.4
- net GND: now also R1.1, R2.2, SV1.39, U3.10, U3.5, U3.7; no longer C1.2, C2.2, C3.2, C4.2, D1.C, U1.1, U1.4, U2.10, U2.5, U2.7
- net INT: now also SV1.7, U3.11; no longer U1.3, U2.11
- net SCL: now also SV1.5, U3.12; no longer U1.5, U2.13
- net SDA: now also SV1.3, U3.13; no longer U1.2, U2.12
- net VCCA: now also R2.1, SV1.1, U3.1; no longer C3.1, U2.1, U2.8
- net VCCB: now also R1.2, SV1.2, U3.14; no longer C4.1, R1.1, U2.14
Routing:
- net VCCB: track 19.8 -> 61.2 mm
- net A2: track 44.7 -> 15.7 mm
- net LED: track 0.00 -> 26.0 mm, vias 0 -> 1
- net N$1: track 0.00 -> 23.8 mm
- net GND: track 2.99 -> 22.9 mm, vias 3 -> 2
- net INT: track 10.2 -> 26.9 mm
- net A1: track 32.7 -> 16.2 mm
- net VCCA: track 41.5 -> 57.6 mm, vias 1 -> 0
- net A3: track 40.5 -> 25.6 mm, vias 1 -> 0
- net LS_VDD: track 11.8 -> 0.00 mm
- net LED_2: track 11.6 -> 0.00 mm
- net SDA: track 10.7 -> 18.6 mm
- net LED_1: track 7.57 -> 0.00 mm
- net SCL: track 23.3 -> 18.8 mm, vias 2 -> 0
Other:
- board size 35 x 22 mm -> 55 x 30 mm
- board text added: "Stress Controller Shield Board v1"

Commit message: Update
Routing:
- net VCCA: track 57.6 -> 88.8 mm
- net VCCB: track 61.2 -> 49.8 mm, vias 0 -> 2
- net INT: track 26.9 -> 21.9 mm
- net SDA: track 18.6 -> 21.7 mm
- net SCL: track 18.8 -> 20.2 mm
Other:
- board size 55 x 30 mm -> 55.4 x 31.3 mm
