File: PCB - EAGLE Files/Models/PCB_1/PCB_Gabri1.1.1.brd (EAGLE design)
At the start: 35 x 22 mm, 10 parts, among them U1 VEML6030, U2 TXS0104ED, X1 0446200002

Commit message: Updating PCB printings
Routing:
- net INT: track 9.85 -> 9.26 mm
- net GND: track 6.03 -> 6.43 mm, vias 4 -> 5
