File: PCB - EAGLE Files/Models/PCB_1_SecondVersion/PCB_Gabri1.1.1.brd (EAGLE design)
At the start: 37 x 24 mm, 10 parts, among them U1 VEML6030, U2 TXS0104ED, X1 0446200002

Commit message: gerber
Routing:
- net A3: track 49.4 -> 47.6 mm
- net A2: track 61.2 -> 62.5 mm
- net GND: vias 4 -> 5
Changed lines of the file:
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@@
 <layer number="18" name="Vias" color="2" fill="1" visible="yes" active="yes"/>
 <layer number="19" name="Unrouted" color="6" fill="1" visible="yes" active="yes"/>
-<layer number="20" name="Dimension" color="15" fill="1" visible="yes" active="yes"/>
+<layer number="20" name="Dimension" color="15" fill="1" visible="no" active="yes"/>
 <layer number="21" name="tPlace" color="7" fill="1" visible="yes" active="yes"/>
 <layer number="22" name="bPlace" color="7" fill="1" visible="no" active="yes"/>
@@
 <param name="mtCopper" value="0.035mm 0.035mm 0.035mm 0.035mm 0.035mm 0.035mm 0.035mm 0.035mm 0.035mm 0.035mm 0.035mm 0.035mm 0.035mm 0.035mm 0.035mm 0.035mm"/>
 <param name="mtIsolate" value="1.5mm 0.15mm 0.2mm 0.15mm 0.2mm 0.15mm 0.2mm 0.15mm 0.2mm 0.15mm 0.2mm 0.15mm 0.2mm 0.15mm 0.2mm"/>
-<param name="mdWireWire" value="0.8mm"/>
-<param name="mdWirePad" value="8mil"/>
-<param name="mdWireVia" value="8mil"/>
+<param name="mdWireWire" value="0.9mm"/>
+<param name="mdWirePad" value="0.9mm"/>
+<param name="mdWireVia" value="0.9mm"/>
 <param name="mdPadPad" value="8mil"/>
 <param name="mdPadVia" value="8mil"/>
@@
 <contactref element="U2" pad="3"/>
 <wire x1="62.06241875" y1="66.3036" x2="61.4436" y2="66.92241875" width="0.4064" layer="1"/>
-<wire x1="93.5101" y1="72.11343125" x2="92.58016875" y2="71.1835" width="0.4064" layer="1"/>
-<wire x1="92.58016875" y1="71.1835" x2="91.26503125" y2="71.1835" width="0.4064" layer="1"/>
 <wire x1="61.4436" y1="66.92241875" x2="61.4436" y2="72.33758125" width="0.4064" layer="1"/>
 <wire x1="61.4436" y1="72.33758125" x2="70.00961875" y2="80.9036" width="0.4064" layer="1"/>
 <wire x1="67.2394" y1="66.09" x2="67.0258" y2="66.3036" width="0.4064" layer="1"/>
 <wire x1="67.0258" y1="66.3036" x2="62.06241875" y2="66.3036" width="0.4064" layer="1"/>
-<wire x1="70.00961875" y1="80.9036" x2="89.13035" y2="80.9036" width="0.4064" layer="1"/>
-<wire x1="89.13035" y1="80.9036" x2="93.5101" y2="76.52385" width="0.4064" layer="1"/>
-<wire x1="93.5101" y1="76.52385" x2="93.5101" y2="72.11343125" width="0.4064" layer="1"/>
-<wire x1="91.26503125" y1="71.1835" x2="90.56653125" y2="71.882" width="0.4064" layer="1"/>
-<wire x1="90.56653125" y1="71.882" x2="86.36" y2="71.882" width="0.4064" layer="1"/>
+<wire x1="89.13035" y1="80.9036" x2="70.00961875" y2="80.9036" width="0.4064" layer="1"/>
+<wire x1="86.36" y1="71.882" x2="89.418" y2="71.882" width="0.4064" layer="1"/>
+<wire x1="89.418" y1="71.882" x2="90.4" y2="70.9" width="0.4064" layer="1"/>
+<wire x1="90.4" y1="70.9" x2="93.1" y2="70.9" width="0.4064" layer="1"/>
+<wire x1="93.1" y1="70.9" x2="94.15" y2="71.95" width="0.4064" layer="1"/>
+<wire x1="94.15" y1="71.95" x2="94.15" y2="75.88395" width="0.4064" layer="1"/>
+<wire x1="94.15" y1="75.88395" x2="89.13035" y2="80.9036" width="0.4064" layer="1"/>
 </signal>
 <signal name="A3">
 <contactref element="U2" pad="4"/>
 <contactref element="X1" pad="3"/>
-<wire x1="85.344" y1="73.66" x2="85.344" y2="78.65" width="0.4064" layer="1"/>
-<wire x1="85.344" y1="78.65" x2="82.25" y2="78.65" width="0.4064" layer="1"/>
-<via x="82.25" y="78.65" extent="1-16" drill="0.6"/>
 <via x="61.15" y="64.75" extent="1-16" drill="0.6"/>
-<wire x1="82.25" y1="78.65" x2="78.68395" y2="78.65" width="0.4064" layer="16"/>
+<wire x1="78.68395" y1="78.65" x2="82.25" y2="78.65" width="0.4064" layer="16"/>
 <wire x1="78.68395" y1="78.65" x2="78.54315" y2="78.7908" width="0.4064" layer="16"/>
 <wire x1="78.54315" y1="78.7908" x2="76.39685" y2="78.7908" width="0.4064" layer="16"/>
@@
 <wire x1="61.15" y1="64.75" x2="67.2394" y2="64.75" width="0.4064" layer="1"/>
 <wire x1="67.2394" y1="64.75" x2="67.2394" y2="64.82" width="0.4064" layer="1"/>
+<wire x1="82.25" y1="78.65" x2="85.05" y2="75.85" width="0.4064" layer="16"/>
+<wire x1="85.05" y1="75.85" x2="85.1" y2="75.85" width="0.4064" layer="16"/>
+<via x="85.1" y="75.85" extent="1-16" drill="0.6"/>
+<wire x1="85.1" y1="75.85" x2="85.344" y2="75.606" width="0.4064" layer="1"/>
+<wire x1="85.344" y1="75.606" x2="85.344" y2="73.66" width="0.4064" layer="1"/>
 </signal>
 <signal name="VCCA">
@@
 <wire x1="70.9832" y1="75.3118875" x2="74.4621125" y2="78.7908" width="0.4064" layer="1"/>
 <wire x1="74.4621125" y1="78.7908" x2="78.54315" y2="78.7908" width="0.4064" layer="1"/>
-<wire x1="82.63395" y1="74.7" x2="82.9" y2="74.7" width="0.4064" layer="1"/>
-<wire x1="78.54315" y1="78.7908" x2="82.63395" y2="74.7" width="0.4064" layer="1"/>
-<wire x1="82.9" y1="74.7" x2="83.312" y2="74.288" width="0.4064" layer="1"/>
-<wire x1="83.312" y1="74.288" x2="83.312" y2="73.66" width="0.4064" layer="1"/>
 <wire x1="72.04" y1="61.01" x2="69.1476375" y2="61.01" width="0.4064" layer="1"/>
 <wire x1="67.453" y1="68.4164" x2="67.2394" y2="68.63" width="0.4064" layer="1"/>
@@
 <wire x1="69.1476375" y1="67.36" x2="68.0912375" y2="68.4164" width="0.4064" layer="1"/>
 <wire x1="68.0912375" y1="68.4164" x2="67.453" y2="68.4164" width="0.4064" layer="1"/>
+<wire x1="78.54315" y1="78.7908" x2="83.312" y2="74.02195" width="0.4064" layer="1"/>
+<wire x1="83.312" y1="74.02195" x2="83.312" y2="73.66" width="0.4064" layer="1"/>
 </signal>
 <signal name="INT">
@@
 </polygon>
 <via x="78.2" y="73.1" extent="1-16" drill="0.5"/>
+<via x="64.55" y="69.7" extent="1-16" drill="0.6"/>
 </signal>
 <signal name="LED_1">
