File: PCB - EAGLE Files/Models/PCB_2/PCB_2.1.brd (EAGLE design)
At the start: 55.4 x 31.3 mm, 6 parts, among them U3 TXS0104ED, X1 0446200002

Commit message: Updating PCB printings
Parts:
- moved R2 2.92 mm to (33.2, 15.4)
- moved U3 2.92 mm to (25.6, 17.9)
- moved R3 2.92 mm to (33.2, 10.3)
- moved R1 2.92 mm to (33.2, 20.5)
- moved SV1 2.92 mm to (26.8, 26.8)
- moved X1 2.92 mm to (2.71, 12.9)
Connections:
- removed net A1: U3.2, X1.1
- removed net A2: U3.3, X1.2
- new net N$2: U3.2, X1.2
- new net N$3: U3.3, X1.1
Routing:
- net GND: track 22.9 -> 2.98 mm, vias 2 -> 3
- net N$3: track 0.00 -> 18.0 mm
- net N$1: track 23.8 -> 40.1 mm
- net A1: track 16.2 -> 0.00 mm
- net A3: track 25.6 -> 41.5 mm
- net A2: track 15.7 -> 0.00 mm
- net N$2: track 0.00 -> 13.7 mm
- net VCCA: track 88.8 -> 90.8 mm
Other:
- board size 55.4 x 31.3 mm -> 63 x 37 mm

Commit message: Uploading gerber files
Connections:
- new net BUZZER: SV1.40
Routing:
- net N$1: track 40.1 -> 46.0 mm
Changed lines of the file:
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@@
 <wire x1="19.2" y1="23.7" x2="19.2" y2="28.9" width="0.508" layer="1"/>
 <wire x1="21.76" y1="17.94" x2="21.76" y2="21.14" width="0.508" layer="1"/>
-<wire x1="21.76" y1="21.14" x2="19.2" y2="23.7" width="0.508" layer="1"/>
+<wire x1="21.76" y1="21.14" x2="20.4" y2="22.5" width="0.508" layer="1"/>
+<wire x1="20.4" y1="22.5" x2="19.2" y2="23.7" width="0.508" layer="1"/>
 </signal>
 <signal name="N$1">
 <contactref element="SV1" pad="37"/>
 <contactref element="R3" pad="2"/>
-<wire x1="34.14" y1="10.32" x2="40.75" y2="10.32" width="0.508" layer="1"/>
-<wire x1="40.75" y1="10.32" x2="53.73" y2="23.3" width="0.508" layer="1"/>
 <wire x1="53.73" y1="23.3" x2="53.73" y2="30.37" width="0.508" layer="1"/>
 <wire x1="53.73" y1="30.37" x2="52.7" y2="31.4" width="0.508" layer="1"/>
 <wire x1="48.43" y1="28.1" x2="48.43" y2="29.83" width="0.508" layer="1"/>
-<wire x1="48.43" y1="29.83" x2="49.7" y2="31.1" width="0.508" layer="1"/>
-<wire x1="49.7" y1="31.1" x2="49.9" y2="31.3" width="0.508" layer="1"/>
+<wire x1="48.43" y1="29.83" x2="50" y2="31.4" width="0.508" layer="1"/>
 <wire x1="52.7" y1="31.4" x2="50" y2="31.4" width="0.508" layer="1"/>
-<wire x1="50" y1="31.4" x2="49.9" y2="31.3" width="0.508" layer="1"/>
+<wire x1="50.82" y1="10.32" x2="53.7" y2="13.2" width="0.508" layer="1"/>
+<wire x1="53.7" y1="13.2" x2="53.7" y2="23.27" width="0.508" layer="1"/>
+<wire x1="53.7" y1="23.27" x2="53.73" y2="23.3" width="0.508" layer="1"/>
+<wire x1="34.14" y1="10.32" x2="50.82" y2="10.32" width="0.508" layer="1"/>
 </signal>
 <signal name="N$2">
@@
 <wire x1="17.0272125" y1="8.6" x2="5.954" y2="8.6" width="0.508" layer="1"/>
 </signal>
+<signal name="BUZZER">
+<contactref element="SV1" pad="40"/>
+</signal>
 </signals>

Commit message: Test
Connections:
- net N$2 renamed A1
- net N$3 renamed A2
Changed lines of the file:
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@@
 <wire x1="34.14" y1="10.32" x2="50.82" y2="10.32" width="0.508" layer="1"/>
 </signal>
-<signal name="N$2">
+<signal name="A1">
 <contactref element="U3" pad="2"/>
 <contactref element="X1" pad="2"/>
@@
 <wire x1="19.179590625" y1="12.460753125" x2="17.0388375" y2="10.32" width="0.508" layer="1"/>
 </signal>
-<signal name="N$3">
+<signal name="A2">
 <contactref element="U3" pad="3"/>
 <contactref element="X1" pad="1"/>
