File: PCB - EAGLE Files/Models/PCB_2/PCB_2.1.sch (EAGLE design)
At the start: 6 parts, among them U3 TXS0104ED, X1 0446200002

Commit message: Test
Connections:
- net N$2 renamed A1
- net N$3 renamed A2
Changed lines of the file:
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@@
 </segment>
 </net>
-<net name="N$2" class="0">
+<net name="A1" class="0">
 <segment>
 <pinref part="U3" gate="A" pin="A1"/>
@@
 </segment>
 </net>
-<net name="N$3" class="0">
+<net name="A2" class="0">
 <segment>
 <pinref part="U3" gate="A" pin="A2"/>
