File: PCB - EAGLE Files/Models/New Version/PCB_RPI/PCB_2.1.brd (EAGLE design)
At the start: 63 x 37 mm, 7 parts, among them X1 0446200002

Commit message: Uploaded printings of final version pcb
Parts:
- removed R1, R4: TCR0805N910K, TCR0805N910K:RESC2012X65N
- removed SG1: F/EE17P, buzzer:F/EE17P
- moved X1 7.67 mm to (9.81, 11.1)
- moved R3 5.19 mm to (29.3, 8.80), turned to 0 degrees
- moved R2 2.85 mm to (29.4, 3.60), turned to 0 degrees
Connections:
- removed net BUZZER: R4.2, SV1.9
- removed net INT: R1.1, SV1.7, X1.4
- removed net N$5: SG1.1, SV1.39, X1.8
- removed net N$6: R4.1, SG1.2
- new net GND: SV1.39, X1.8
- new net N$1: X1.4
- net 3V3: no longer R1.2
Routing:
- net 3V3: track 17.0 -> 104.6 mm, vias 0 -> 1
- net SCL: track 0.00 -> 67.1 mm, vias 0 -> 1
- net SDA: track 0.00 -> 57.5 mm, vias 0 -> 2
- net GND: track 0.00 -> 45.2 mm, vias 0 -> 2
- net INT: track 35.1 -> 0.00 mm
- net BUZZER: track 30.4 -> 0.00 mm
- net N$6: track 16.8 -> 0.00 mm
